Commit message: Place the steering limits asymmetrically at -280/+100 degrees
A wheel direction is periodic modulo 180 degrees, so mechanical travel only
fixes the guaranteed margin -- every direction has a branch with margin m iff
the span is at least 180+2m, and 380 degrees of travel already buys the maximum
m = 100. What the placement decides is which direction is left owning the branch
that sits beside a limit. Symmetric +-190 put that branch on straight ahead,
where 180 degrees had 10 degrees of margin and was held for a whole 110 s pass;
that is what cost a 100 m pass a 180 degree reconfiguration 15 mm from its end.
[-280, +100] leaves it on lateral +90 instead, held only during a 6-10 s
transfer, and gives both straight-ahead branches 95 degrees.

All four corners keep one pair of limits. A left/right mirror was measured
against the run data and rejected: in-place rotation pairs the wheels by
diagonal (fl/rr against fr/rl), so a left/right mirror does not align with its
symmetry and only permutes which two wheels sit at the smaller margin; lateral
motion wants all four wheels at one angle, so mirroring would reintroduce the
front/rear split that one shared pair removes, and it would make the corner
modules handed on a real vehicle.

Config::soft becomes soft_lower/soft_upper plus derived span(), margin() and
recentre_margin(); the five uses follow. Only limit_approach changes meaning:
with the limits off centre, "moving away from zero" is no longer "moving toward
a limit", so it now takes the sign of the motion and the headroom left on that
side. validate() replaces the per-endpoint checks a symmetric limit needed with
the span relation, which already guarantees a legal lateral branch.

Travel stays 380 degrees and the 8 degree mechanical reserve is untouched, so
cable wrap is unchanged; the mechanical zero is no longer mid-travel, which a
real vehicle's homing and assembly datum would have to account for.

Measured: the three spin-recovery cases all return to straight in 54.13 degrees
with 95 degrees of margin, and the 126 degree recentring the segment margin had
reintroduced is gone. A 7-pass 13 m mission at 1.0 m/s reached ACQUIRED in 321 s
with RTF 0.9986, 63 blocks, zero LIMIT_RECONFIGURE, and steering dwelling only
at -125.9, -54.1, 0 and -180 degrees; least margin over the run was 16.01
degrees on a transfer transient. 329 tests pass. The tail-coverage NEEDS_RESCAN
is unrelated and still open.

Co-Authored-By: Claude Opus 5 <noreply@anthropic.com>
Claude-Session: https://claude.ai/code/session_01V4VVKBt9dtBDDnco8GRjYV

File: src/agv_description/urdf/agv.urdf.xacro (robot description, xacro)
@@ -134,5 +134,5 @@
     <joint name="${name}_steer_joint" type="revolute"><parent link="${name}_suspension_link"/><child link="${name}_steer_link"/>
       <origin xyz="0 0 -0.10"/><axis xyz="0 0 1"/>
-      <limit lower="${-p.steer_hard_limit}" upper="${p.steer_hard_limit}" effort="${p.steer_effort}" velocity="${p.steer_rate}"/>
+      <limit lower="${p.steer_hard_lower}" upper="${p.steer_hard_upper}" effort="${p.steer_effort}" velocity="${p.steer_rate}"/>
       <dynamics damping="0.5" friction="0.1"/>
     </joint>
@@ -196,5 +196,5 @@
   <ros2_control name="GazeboSystem" type="system"><hardware><plugin>gz_ros2_control/GazeboSimSystem</plugin></hardware>
     <xacro:macro name="interfaces" params="name">
-      <joint name="${name}_steer_joint"><command_interface name="position"><param name="min">${-p.steer_hard_limit}</param><param name="max">${p.steer_hard_limit}</param></command_interface><state_interface name="position"/><state_interface name="velocity"/></joint>
+      <joint name="${name}_steer_joint"><command_interface name="position"><param name="min">${p.steer_hard_lower}</param><param name="max">${p.steer_hard_upper}</param></command_interface><state_interface name="position"/><state_interface name="velocity"/></joint>
       <joint name="${name}_drive_joint"><command_interface name="velocity"><param name="min">${-p.max_speed/p.wheel_radius}</param><param name="max">${p.max_speed/p.wheel_radius}</param></command_interface><state_interface name="position"/><state_interface name="velocity"/></joint>
     </xacro:macro>
