Commit message: Model wheel-shaft encoder triggers and independent physical tyre diameter

File: src/agv_description/urdf/agv.urdf.xacro (robot description, xacro)
@@ -3,5 +3,9 @@
   <xacro:arg name="platform" default="$(find agv_description)/config/platform.yaml"/>
   <xacro:arg name="controllers" default="$(find agv_bringup)/config/controllers.yaml"/>
+  <xacro:arg name="actual_wheel_diameter" default="0"/>
   <xacro:property name="p" value="${xacro.load_yaml('$(arg platform)')}"/>
+  <!-- Physical tyre only; control/odometry retain platform.wheel_radius. -->
+  <xacro:property name="actual_diameter" value="${float('$(arg actual_wheel_diameter)')}"/>
+  <xacro:property name="physical_radius" value="${actual_diameter/2 if actual_diameter > 0 else p.wheel_radius}"/>
   <xacro:arg name="camera_config" default="$(find agv_description)/config/linescan.yaml"/>
   <xacro:property name="cam" value="${xacro.load_yaml('$(arg camera_config)')}"/>
@@ -101,5 +105,5 @@
   <xacro:macro name="tread" params="i">
     <xacro:if value="${i &lt; 24}">
-      <visual><origin xyz="${(p.wheel_radius-.004)*sin(i*pi/12)} 0 ${(p.wheel_radius-.004)*cos(i*pi/12)}" rpy="0 ${i*pi/12} 0"/><geometry><box size="0.038 ${p.wheel_width*.86} 0.008"/></geometry><material name="tire"/></visual>
+      <visual><origin xyz="${(physical_radius-.004)*sin(i*pi/12)} 0 ${(physical_radius-.004)*cos(i*pi/12)}" rpy="0 ${i*pi/12} 0"/><geometry><box size="0.038 ${p.wheel_width*.86} 0.008"/></geometry><material name="tire"/></visual>
       <xacro:tread i="${i+1}"/>
     </xacro:if>
@@ -138,8 +142,8 @@
     </joint>
     <link name="${name}_wheel_link">
-      <inertial><mass value="18.0"/><inertia ixx="${18*(3*p.wheel_radius**2+p.wheel_width**2)/12}" iyy="${18*p.wheel_radius**2/2}" izz="${18*(3*p.wheel_radius**2+p.wheel_width**2)/12}" ixy="0" ixz="0" iyz="0"/></inertial>
+      <inertial><mass value="18.0"/><inertia ixx="${18*(3*physical_radius**2+p.wheel_width**2)/12}" iyy="${18*physical_radius**2/2}" izz="${18*(3*physical_radius**2+p.wheel_width**2)/12}" ixy="0" ixz="0" iyz="0"/></inertial>
       <xacro:tread i="${0}"/>
-      <visual><origin rpy="${pi/2} 0 0"/><geometry><cylinder radius="${p.wheel_radius-.006}" length="${p.wheel_width}"/></geometry><material name="tire"/></visual>
-      <collision><origin rpy="${pi/2} 0 0"/><geometry><cylinder radius="${p.wheel_radius}" length="${p.wheel_width}"/></geometry></collision>
+      <visual><origin rpy="${pi/2} 0 0"/><geometry><cylinder radius="${physical_radius-.006}" length="${p.wheel_width}"/></geometry><material name="tire"/></visual>
+      <collision><origin rpy="${pi/2} 0 0"/><geometry><cylinder radius="${physical_radius}" length="${p.wheel_width}"/></geometry></collision>
       <visual><origin xyz="0 ${p.wheel_width/2+0.002} 0" rpy="${pi/2} 0 0"/><geometry><cylinder radius="0.085" length="0.006"/></geometry><material name="metal"/></visual>
       <visual><origin xyz="0 ${-p.wheel_width/2-0.002} 0" rpy="${pi/2} 0 0"/><geometry><cylinder radius="0.085" length="0.006"/></geometry><material name="metal"/></visual>

Commit message: Add passive camera bracket flex and sample its physical pose

File: src/agv_description/urdf/agv.urdf.xacro (robot description, xacro)
@@ -11,4 +11,6 @@
   <xacro:property name="cam" value="${xacro.load_yaml('$(arg camera_config)')}"/>
   <xacro:property name="camera_height" value="${cam.nominal_width_m*cam.focal_length_m/(cam.width*cam.pixel_pitch_m)}"/>
+  <xacro:property name="flex" value="${cam.get('mount_flex', dict(enabled=False))}"/>
+  <xacro:property name="flexible" value="${flex.get('enabled',False)}"/>
   <xacro:property name="lid" value="${xacro.load_yaml('$(find agv_description)/config/lidar.yaml')}"/>
   <material name="orange"><color rgba="1 0.23 0.025 1"/></material>
@@ -25,5 +27,5 @@
   <!-- Large 550 kg AGV; base_link nominally 0.65m above ground. Battery is low. -->
   <link name="base_link">
-    <xacro:box_inertia m="${p.mass-337.2}" x="1.90" y="1.10" z="0.50"/>
+    <xacro:box_inertia m="${p.mass-340.2}" x="1.90" y="1.10" z="0.50"/>
     <visual><geometry><mesh filename="file://$(find agv_description)/meshes/large_body.obj"/></geometry><material name="orange"/></visual>
     <collision><geometry><mesh filename="file://$(find agv_description)/meshes/large_body.obj"/></geometry></collision>
@@ -53,8 +55,4 @@
       <xacro:box_visual x="0.08" y="0.08" z="0.12" xyz="0.97 ${y} 0.15" rpy="0 0 0" color="white"/>
       <collision><origin xyz="0.97 ${y} 0.15"/><geometry><box size="0.08 0.08 0.12"/></geometry></collision>
-      <xacro:box_visual x="0.04" y="0.04" z="0.30" xyz="1.005 ${y} 0.29" rpy="0 0 0" color="white"/>
-      <collision><origin xyz="1.005 ${y} 0.29"/><geometry><box size="0.04 0.04 0.30"/></geometry></collision>
-      <xacro:box_visual x="0.17" y="0.035" z="0.035" xyz="1.065 ${y} 0.44" rpy="0 0 0" color="white"/>
-      <collision><origin xyz="1.065 ${y} 0.44"/><geometry><box size="0.17 0.035 0.035"/></geometry></collision>
       <xacro:box_visual x="0.04" y="0.04" z="${0.81-(cam.led_height_m+0.035)}" xyz="0.94 ${y} ${(0.81+cam.led_height_m+0.035)/2-cam.base_nominal_height_m}" rpy="0 0 0" color="metal"/>
       <collision><origin xyz="0.94 ${y} ${(0.81+cam.led_height_m+0.035)/2-cam.base_nominal_height_m}"/><geometry><box size="0.04 0.04 ${0.81-(cam.led_height_m+0.035)}"/></geometry></collision>
@@ -63,5 +61,4 @@
     </xacro:macro>
     <xacro:front_arm y="0.24"/><xacro:front_arm y="-0.24"/>
-    <xacro:box_visual x="0.05" y="0.54" z="0.03" xyz="1.10 0 0.44" rpy="0 0 0" color="white"/>
     <visual><origin xyz="0 0 0.48"/><geometry><cylinder radius="0.04" length="0.05"/></geometry><material name="orange"/></visual>
   </link>
@@ -159,5 +156,35 @@
   <!-- Nominal optics geometry; the visible LED uses overlapping, shadow-casting spot lights. -->
   <link name="camera_link"><xacro:box_inertia m="1.0" x="0.10" y="0.12" z="0.08"/><xacro:box_visual x="0.10" y="0.12" z="0.08" xyz="0 0 0" rpy="0 0 0" color="metal"/><collision><geometry><box size="0.10 0.12 0.08"/></geometry></collision></link>
-  <joint name="camera_mount" type="fixed"><parent link="base_link"/><child link="camera_link"/><origin xyz="${cam.camera_x_m} 0 ${camera_height-cam.base_nominal_height_m+0.04}"/></joint>
+  <!-- Two equivalent bending modes of the upper bracket. Physical springs,
+       no prescribed pose/noise. LED arms and lower mounting blocks stay rigid. -->
+    <link name="camera_roll_link"><xacro:box_inertia m="0.1" x="0.08" y="0.54" z="0.02"/></link>
+    <joint name="camera_roll_joint" type="${'revolute' if flexible else 'fixed'}">
+      <parent link="base_link"/><child link="camera_roll_link"/><origin xyz="1.005 0 0.14"/><axis xyz="1 0 0"/>
+      <limit lower="-0.0872664626" upper="0.0872664626" effort="1000" velocity="5"/>
+      <dynamics damping="${flex.get('damping_nms_rad',5.0)}"/>
+    </joint>
+    <xacro:if value="${flexible}"><gazebo reference="camera_roll_joint"><springStiffness>${flex['stiffness_nm_rad']}</springStiffness><springReference>0</springReference></gazebo></xacro:if>
+    <link name="camera_carrier_link">
+      <inertial><origin xyz="0.07 0 0.15"/><mass value="2.9"/>
+        <inertia ixx="${2.9*(.54**2+.30**2)/12}" iyy="${2.9*(.17**2+.30**2)/12}" izz="${2.9*(.17**2+.54**2)/12}" ixy="0" ixz="0" iyz="0"/>
+      </inertial>
+      <xacro:macro name="moving_arm" params="y">
+        <xacro:box_visual x="0.04" y="0.04" z="0.30" xyz="0 ${y} 0.15" rpy="0 0 0" color="white"/>
+        <collision><origin xyz="0 ${y} 0.15"/><geometry><box size="0.04 0.04 0.30"/></geometry></collision>
+        <xacro:box_visual x="0.17" y="0.035" z="0.035" xyz="0.06 ${y} 0.30" rpy="0 0 0" color="white"/>
+        <collision><origin xyz="0.06 ${y} 0.30"/><geometry><box size="0.17 0.035 0.035"/></geometry></collision>
+      </xacro:macro>
+      <xacro:moving_arm y="0.24"/><xacro:moving_arm y="-0.24"/>
+      <xacro:box_visual x="0.05" y="0.54" z="0.03" xyz="0.095 0 0.30" rpy="0 0 0" color="white"/>
+    </link>
+    <joint name="camera_pitch_joint" type="${'revolute' if flexible else 'fixed'}">
+      <parent link="camera_roll_link"/><child link="camera_carrier_link"/><axis xyz="0 1 0"/>
+      <limit lower="-0.0872664626" upper="0.0872664626" effort="1000" velocity="5"/>
+      <dynamics damping="${flex.get('damping_nms_rad',5.0)}"/>
+    </joint>
+    <!-- Balance gravity at the nominal level pose, not an added oscillation.
+         Camera mass 1 kg + carrier 2.9 kg; roll has symmetric loading. -->
+    <xacro:if value="${flexible}"><gazebo reference="camera_pitch_joint"><springStiffness>${flex['stiffness_nm_rad']}</springStiffness><springReference>${-9.81*(2.9*.07+cam.camera_x_m-1.005)/flex['stiffness_nm_rad']}</springReference></gazebo></xacro:if>
+    <joint name="camera_mount" type="fixed"><parent link="camera_carrier_link"/><child link="camera_link"/><origin xyz="${cam.camera_x_m-1.005} 0 ${camera_height-cam.base_nominal_height_m+0.04-.14}"/></joint>
   <link name="camera_optical_frame"/>
   <joint name="camera_optical_joint" type="fixed"><parent link="camera_link"/><child link="camera_optical_frame"/><origin xyz="0 0 -0.04" rpy="${pi} 0 ${pi/2}"/></joint>
@@ -205,4 +232,8 @@
     <xacro:macro name="passive" params="name"><joint name="${name}_suspension_joint"><state_interface name="position"/><state_interface name="velocity"/></joint></xacro:macro>
     <xacro:passive name="fl"/><xacro:passive name="fr"/><xacro:passive name="rl"/><xacro:passive name="rr"/>
+    <xacro:if value="${flexible}">
+      <joint name="camera_roll_joint"><state_interface name="position"/><state_interface name="velocity"/></joint>
+      <joint name="camera_pitch_joint"><state_interface name="position"/><state_interface name="velocity"/></joint>
+    </xacro:if>
     <xacro:interfaces name="fl"/><xacro:interfaces name="fr"/><xacro:interfaces name="rl"/><xacro:interfaces name="rr"/>
   </ros2_control>

Commit message: Share camera mount pivot across model and sensor

File: src/agv_description/urdf/agv.urdf.xacro (robot description, xacro)
@@ -13,4 +13,7 @@
   <xacro:property name="flex" value="${cam.get('mount_flex', dict(enabled=False))}"/>
   <xacro:property name="flexible" value="${flex.get('enabled',False)}"/>
+  <xacro:property name="camera_mass" value="${1.0}"/>
+  <xacro:property name="camera_carrier_mass" value="${2.9}"/>
+  <xacro:property name="camera_carrier_com_x" value="${0.07}"/>
   <xacro:property name="lid" value="${xacro.load_yaml('$(find agv_description)/config/lidar.yaml')}"/>
   <material name="orange"><color rgba="1 0.23 0.025 1"/></material>
@@ -155,10 +158,10 @@
   <xacro:wheel name="rr" x="${-p.wheelbase/2}" y="${-p.track/2}"/>
   <!-- Nominal optics geometry; the visible LED uses overlapping, shadow-casting spot lights. -->
-  <link name="camera_link"><xacro:box_inertia m="1.0" x="0.10" y="0.12" z="0.08"/><xacro:box_visual x="0.10" y="0.12" z="0.08" xyz="0 0 0" rpy="0 0 0" color="metal"/><collision><geometry><box size="0.10 0.12 0.08"/></geometry></collision></link>
+  <link name="camera_link"><xacro:box_inertia m="${camera_mass}" x="0.10" y="0.12" z="0.08"/><xacro:box_visual x="0.10" y="0.12" z="0.08" xyz="0 0 0" rpy="0 0 0" color="metal"/><collision><geometry><box size="0.10 0.12 0.08"/></geometry></collision></link>
   <!-- Two equivalent bending modes of the upper bracket. Physical springs,
        no prescribed pose/noise. LED arms and lower mounting blocks stay rigid. -->
     <link name="camera_roll_link"><xacro:box_inertia m="0.1" x="0.08" y="0.54" z="0.02"/></link>
     <joint name="camera_roll_joint" type="${'revolute' if flexible else 'fixed'}">
-      <parent link="base_link"/><child link="camera_roll_link"/><origin xyz="1.005 0 0.14"/><axis xyz="1 0 0"/>
+      <parent link="base_link"/><child link="camera_roll_link"/><origin xyz="${flex['pivot_x_m']} 0 ${flex['pivot_z_m']}"/><axis xyz="1 0 0"/>
       <limit lower="-0.0872664626" upper="0.0872664626" effort="1000" velocity="5"/>
       <dynamics damping="${flex.get('damping_nms_rad',5.0)}"/>
@@ -166,6 +169,6 @@
     <xacro:if value="${flexible}"><gazebo reference="camera_roll_joint"><springStiffness>${flex['stiffness_nm_rad']}</springStiffness><springReference>0</springReference></gazebo></xacro:if>
     <link name="camera_carrier_link">
-      <inertial><origin xyz="0.07 0 0.15"/><mass value="2.9"/>
-        <inertia ixx="${2.9*(.54**2+.30**2)/12}" iyy="${2.9*(.17**2+.30**2)/12}" izz="${2.9*(.17**2+.54**2)/12}" ixy="0" ixz="0" iyz="0"/>
+      <inertial><origin xyz="${camera_carrier_com_x} 0 0.15"/><mass value="${camera_carrier_mass}"/>
+        <inertia ixx="${camera_carrier_mass*(.54**2+.30**2)/12}" iyy="${camera_carrier_mass*(.17**2+.30**2)/12}" izz="${camera_carrier_mass*(.17**2+.54**2)/12}" ixy="0" ixz="0" iyz="0"/>
       </inertial>
       <xacro:macro name="moving_arm" params="y">
@@ -184,7 +187,7 @@
     </joint>
     <!-- Balance gravity at the nominal level pose, not an added oscillation.
-         Camera mass 1 kg + carrier 2.9 kg; roll has symmetric loading. -->
-    <xacro:if value="${flexible}"><gazebo reference="camera_pitch_joint"><springStiffness>${flex['stiffness_nm_rad']}</springStiffness><springReference>${-9.81*(2.9*.07+cam.camera_x_m-1.005)/flex['stiffness_nm_rad']}</springReference></gazebo></xacro:if>
-    <joint name="camera_mount" type="fixed"><parent link="camera_carrier_link"/><child link="camera_link"/><origin xyz="${cam.camera_x_m-1.005} 0 ${camera_height-cam.base_nominal_height_m+0.04-.14}"/></joint>
+         Camera and carrier mass properties above also define this preload. -->
+    <xacro:if value="${flexible}"><gazebo reference="camera_pitch_joint"><springStiffness>${flex['stiffness_nm_rad']}</springStiffness><springReference>${-9.81*(camera_carrier_mass*camera_carrier_com_x+camera_mass*(cam.camera_x_m-flex['pivot_x_m']))/flex['stiffness_nm_rad']}</springReference></gazebo></xacro:if>
+    <joint name="camera_mount" type="fixed"><parent link="camera_carrier_link"/><child link="camera_link"/><origin xyz="${cam.camera_x_m-flex['pivot_x_m']} 0 ${camera_height-cam.base_nominal_height_m+0.04-flex['pivot_z_m']}"/></joint>
   <link name="camera_optical_frame"/>
   <joint name="camera_optical_joint" type="fixed"><parent link="camera_link"/><child link="camera_optical_frame"/><origin xyz="0 0 -0.04" rpy="${pi} 0 ${pi/2}"/></joint>

Commit message: Record wheel contact evidence for scan faults

File: src/agv_description/urdf/agv.urdf.xacro (robot description, xacro)
@@ -151,5 +151,14 @@
     <joint name="${name}_drive_joint" type="continuous"><parent link="${name}_steer_link"/><child link="${name}_wheel_link"/>
       <origin xyz="0 0 -0.20"/><axis xyz="0 1 0"/><limit effort="${p.drive_effort}" velocity="${p.max_speed/p.wheel_radius}"/><dynamics damping="0.02"/></joint>
-    <gazebo reference="${name}_wheel_link"><mu1>0.8</mu1><mu2>0.8</mu2><kp>1000000</kp><kd>100</kd></gazebo>
+    <gazebo reference="${name}_wheel_link">
+      <mu1>0.8</mu1><mu2>0.8</mu2><kp>1000000</kp><kd>100</kd>
+      <!-- Per-physics-step evidence for rare wheel / triangle-mesh impulses. The
+           line-scan plugin reads the GZ component into a bounded RAM ring and
+           adds no ROS stream or normal-path disk writes. -->
+      <sensor name="${name}_wheel_contact" type="contact">
+        <always_on>true</always_on><update_rate>1000</update_rate>
+        <contact><collision>${name}_wheel_link_collision</collision></contact>
+      </sensor>
+    </gazebo>
   </xacro:macro>
   <xacro:wheel name="fl" x="${p.wheelbase/2}" y="${p.track/2}"/>
